Commit message: Add FR3 real robot bringup and gripper integration

File: fairino3_v6_moveit2_config/config/fairino3_v6_robot.ros2_control.xacro (robot description, xacro)
@@ -44,4 +44,10 @@
                 </state_interface>
             </joint>
+            <joint name="gripper_joint">
+                <command_interface name="position"/>
+                <state_interface name="position">
+                  <param name="initial_value">${initial_positions['gripper_joint']}</param>
+                </state_interface>
+            </joint>
         </ros2_control>
     </xacro:macro>

File: fairino3_v6_moveit2_config/config/fairino3_v6_robot.urdf.xacro (robot description, xacro)
@@ -1,9 +1,21 @@
 <?xml version="1.0"?>
-<robot xmlns:xacro="http://www.ros.org/wiki/xacro" name="fairino3_v6_robot">
-    <xacro:arg name="initial_positions_file" default="initial_positions.yaml" />
-    <!-- Import fairino3_v6_robot urdf file -->
-    <xacro:include filename="$(find fairino_description)/urdf/fairino3_v6.urdf" />
-    <!-- Import control_xacro -->
-    <xacro:include filename="fairino3_v6_robot.ros2_control.xacro" />
-    <xacro:fairino3_v6_robot_ros2_control name="FakeSystem" initial_positions_file="$(arg initial_positions_file)"/>
+<robot xmlns:xacro="http://www.ros.org/wiki/xacro"
+       name="fairino3_v6_robot">
+  <xacro:arg
+      name="initial_positions_file"
+      default="initial_positions.yaml" />
+  <!-- FR3 robot -->
+  <xacro:include
+      filename="$(find fairino_description)/urdf/fairino3_v6.urdf" />
+  <!-- HKV TG-9801 真夹爪：安装面贴紧 wrist3 法兰并对中 -->
+  <xacro:include
+      filename="$(find fairino_description)/urdf/hkv_gripper.xacro" />
+  <xacro:hkv_gripper
+      parent="wrist3_link" />
+  <!-- ros2_control -->
+  <xacro:include
+      filename="fairino3_v6_robot.ros2_control.xacro" />
+  <xacro:fairino3_v6_robot_ros2_control
+      name="FakeSystem"
+      initial_positions_file="$(arg initial_positions_file)"/>
 </robot>
