Commit message: update_simpose

File: fairino_description/urdf/hkv_gripper.xacro (robot description, xacro)
@@ -364,5 +364,5 @@
     <!-- ======================================================= -->
     <!--
-      修改后的夹爪长度关系：
+      gripper_tcp = 两根夹指最末端之间的中心。
       滑块位置：
           z = 0.070 m
@@ -377,20 +377,11 @@
         = 0.1497 m
         ≈ 0.150 m
-      TCP 仍然保持在两指工作区中部。
-      原来：
-          0.067 + 0.008 + 0.036
-          = 0.111 m
-      修改后：
-          0.070 + 0.008 + 0.036
-          = 0.114 m
-      所以：
-      法兰面 -> TCP
-          ≈ 114 mm
+      法兰面（gripper_base_link）-> TCP
+          = 0.150 m
       法兰面 -> 夹爪最末端
-          ≈ 150 mm
-      如果以后你希望 TCP 就在真正指尖，
-      可以把下面的 z="0.114"
-      改为：
-          z="0.150"
+          ≈ 0.150 m
+      旧定义把 TCP 放在工作区中部（z=0.114），
+      指尖补偿 fingertip_from_tcp=0.036。
+      新定义不再做指尖补偿。
     -->
     <link name="gripper_tcp"/>
@@ -400,10 +391,10 @@
       <!--
         修改前：
-        z = 0.111
+        z = 0.114（工作区中部）
         修改后：
-        z = 0.114
-      -->
-      <origin
-          xyz="0 0 0.114"
+        z = 0.150（两指最末端中心）
+      -->
+      <origin
+          xyz="0 0 0.150"
           rpy="0 0 0"/>
     </joint>
